Commit message: modify urdf,  add and modify launch files

File: urdf/rccn_east_robot_macro.xacro (robot description, xacro)
@@ -3,5 +3,5 @@
         <xacro:macro name="rccn_east_robot" params="prefix">
             <xacro:property name="east_prefix" value="east_" />
-            <xacro:include filename="$(find kuka_kr300_support)/urdf/kr300r2500pro_macro.xacro" />
+            <xacro:include filename="$(find kuka_kr300_support)/urdf/kr300r2500ultra_macro.xacro" />
             <link name="${prefix}east_e1_rail">
                 <visual>
@@ -49,6 +49,6 @@
                 <origin xyz="-0.00206000 -0.00032000 -0.00000000" rpy="-0.00000002 -0.00012841 0.00024798" />
             </joint>
-            <!-- kuka kr300 r2500 pro -->
-            <xacro:kuka_kr300r2500pro prefix="${east_prefix}"/>
+            <!-- kuka kr300 r2500 ultra -->
+            <xacro:kuka_kr300r2500ultra prefix="${east_prefix}"/>
         </xacro:macro>
     </robot>

File: urdf/rccn_kuka_robot_cell.urdf (robot description, URDF)
Before this commit: robot rccn_kuka_robot_cell, 21 links, 20 joints
Links:
- link east_base_link: geometry collision mesh filename=package://kuka_kr300_support/meshes/kr300r2500ultra/collisi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; visual mesh filename=package://kuka_kr300_support/meshes/kr300r2500ultra/visual/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
- link east_link_1: geometry collision mesh filename=package://kuka_kr300_support/meshes/kr300r2500ultra/collisi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; visual mesh filename=package://kuka_kr300_support/meshes/kr300r2500ultra/visual/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
- link east_link_2: geometry collision mesh filename=package://kuka_kr300_support/meshes/kr300r2500ultra/collisi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; visual mesh filename=package://kuka_kr300_support/meshes/kr300r2500ultra/visual/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
- link east_link_3: geometry collision mesh filename=package://kuka_kr300_support/meshes/kr300r2500ultra/collisi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; visual mesh filename=package://kuka_kr300_support/meshes/kr300r2500ultra/visual/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
- link east_link_4: geometry collision mesh filename=package://kuka_kr300_support/meshes/kr300r2500ultra/collisi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; visual mesh filename=package://kuka_kr300_support/meshes/kr300r2500ultra/visual/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
- link east_link_5: geometry collision mesh filename=package://kuka_kr300_support/meshes/kr300r2500ultra/collisi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; visual mesh filename=package://kuka_kr300_support/meshes/kr300r2500ultra/visual/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
- link east_link_6: geometry collision mesh filename=package://kuka_kr300_support/meshes/kr300r2500ultra/collisi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; visual mesh filename=package://kuka_kr300_support/meshes/kr300r2500ultra/visual/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
- link west_base_link: geometry collision mesh filename=package://kuka_kr300_support/meshes/kr300r2500ultra/collisi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; visual mesh filename=package://kuka_kr300_support/meshes/kr300r2500ultra/visual/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
- link west_link_1: geometry collision mesh filename=package://kuka_kr300_support/meshes/kr300r2500ultra/collisi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; visual mesh filename=package://kuka_kr300_support/meshes/kr300r2500ultra/visual/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
- link west_link_2: geometry collision mesh filename=package://kuka_kr300_support/meshes/kr300r2500ultra/collisi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; visual mesh filename=package://kuka_kr300_support/meshes/kr300r2500ultra/visual/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
- link west_link_3: geometry collision mesh filename=package://kuka_kr300_support/meshes/kr300r2500ultra/collisi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; visual mesh filename=package://kuka_kr300_support/meshes/kr300r2500ultra/visual/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
- link west_link_4: geometry collision mesh filename=package://kuka_kr300_support/meshes/kr300r2500ultra/collisi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; visual mesh filename=package://kuka_kr300_support/meshes/kr300r2500ultra/visual/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
- link west_link_5: geometry collision mesh filename=package://kuka_kr300_support/meshes/kr300r2500ultra/collisi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; visual mesh filename=package://kuka_kr300_support/meshes/kr300r2500ultra/visual/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
- link west_link_6: geometry collision mesh filename=package://kuka_kr300_support/meshes/kr300r2500ultra/collisi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; visual mesh filename=package://kuka_kr300_support/meshes/kr300r2500ultra/visual/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

File: urdf/rccn_west_robot_macro.xacro (robot description, xacro)
@@ -3,5 +3,5 @@
         <xacro:macro name="rccn_west_robot" params="prefix">
             <xacro:property name="west_prefix" value="west_" />
-            <xacro:include filename="$(find kuka_kr300_support)/urdf/kr300r2500pro_macro.xacro" />
+            <xacro:include filename="$(find kuka_kr300_support)/urdf/kr300r2500ultra_macro.xacro" />
             <link name="${prefix}west_e1_rail">
                 <visual>
@@ -49,6 +49,6 @@
                 <origin xyz="-0.00043000 -0.00044000 -0.00000000" rpy="0.00000184 0.00009015 0.00206101" />
             </joint>
-            <!-- kuka kr300 r2500 pro -->
-            <xacro:kuka_kr300r2500pro prefix="${west_prefix}"/>
+            <!-- kuka kr300 r2500 ultra -->
+            <xacro:kuka_kr300r2500ultra prefix="${west_prefix}"/>
         </xacro:macro>
     </robot>
